File: demo.kicad_pcb (KiCad board)
At the start: 2 copper layers, 110 x 100 mm, 34 parts, among them J1 Conn_01x02, J2 Conn_01x04, J3 Conn_01x07

Commit message: uodated pcb with sender
Parts:
- removed C3: CP_Radial_D6.3mm_P2.50mm, PCM_Capacitor_THT_AKL:CP_Radial_D6.3mm_P2.50mm
- C2: value C_Disc_D3.8mm_W2.6mm_P2.50mm -> C_Disc_D5.0mm_W2.5mm_P2.50mm; footprint PCM_Capacitor_THT_AKL:C_Disc_D3.8mm_W2.6mm_P2.50mm -> PCM_Capacitor_THT_AKL:C_Disc_D5.0mm_W2.5mm_P2.50mm
Connections:
- net Net-(DOIT1-EN) renamed EN
- R8 pad 1: Net-(RST_LORA1-Pin_2) -> /RST_LORA
- RST_LORA1 pad 1: /RST_LORA -> GND
- RST_LORA1 pad 2: Net-(RST_LORA1-Pin_2) -> /RST_LORA
Routing:
- net GND: track 49.1 -> 117.3 mm
- net Net-(RST_LORA1-Pin_2): track 6.15 -> 0.00 mm
- net +3.3V: track 381.8 -> 379.7 mm
- net /RST_LORA: track 21.7 -> 23.2 mm
