File: demo.kicad_sch (KiCad schematic)
At the start: 34 parts, among them J1 Conn_01x02, J2 Conn_01x04, J3 Conn_01x07

Commit message: uodated pcb with sender
Parts:
- removed C2: C_Disc_D3.8mm_W2.6mm_P2.50mm, PCM_Capacitor_THT_AKL:C_Disc_D3.8mm_W2.6mm_P2.50mm, symbol PCM_Capacitor_AKL:C_Disc_D3.8mm_W2.6mm_P2.50mm
- removed C3: CP_Radial_D6.3mm_P2.50mm, PCM_Capacitor_THT_AKL:CP_Radial_D6.3mm_P2.50mm, symbol PCM_Capacitor_AKL:CP_Radial_D6.3mm_P2.50mm
- added C2: C_Disc_D5.0mm_W2.5mm_P2.50mm, PCM_Capacitor_THT_AKL:C_Disc_D5.0mm_W2.5mm_P2.50mm, symbol PCM_Capacitor_AKL:C_Disc_D5.0mm_W2.5mm_P2.50mm
Connections:
- net GND: now also RST_LORA1.1 (Pin_1), C2.2
- net RST_LORA: now also R8.1, RST_LORA1.2 (Pin_2); no longer RST_LORA1.1 (Pin_1)
- net EN: now reaches DOIT1.16 (EN), J1.2 (Pin_2), R5.1
- net EN: now also C2.1
Other:
- moved on the sheet: J1, R5
