File: demo.kicad_sch (KiCad schematic)
At the start: 30 parts, among them J1 Conn_01x02, J2 Conn_01x04

Commit message: latest update
Parts:
- removed 5vJ1, RST_LORA1: Conn_01x02, Connector_JST:JST_XH_B2B-XH-A_1x02_P2.50mm_Vertical, symbol Connector_Generic:Conn_01x02
- removed J2: Conn_01x04, Connector_PinHeader_2.54mm:PinHeader_1x04_P2.54mm_Vertical, symbol Connector_Generic:Conn_01x04
- removed R8: 1K, LR0204F2K2:RESAD640W45L370D200, symbol LR0204F2K2:LR0204F2K2
- removed SLED1: Conn_01x02, Connector_JST:JST_EH_B2B-EH-A_1x02_P2.50mm_Vertical, symbol Connector_Generic:Conn_01x02
- added C3: CP_Radial_D6.3mm_P2.50mm, PCM_Capacitor_THT_AKL:CP_Radial_D6.3mm_P2.50mm, symbol PCM_Capacitor_AKL:CP_Radial_D6.3mm_P2.50mm
- added J2: JST_07, Connector_PinHeader_2.54mm:PinHeader_1x07_P2.54mm_Vertical, symbol PCM_SL_Connectors:JST_07
- added J3, J4: JST_02, Connector_JST:JST_EH_B2B-EH-A_1x02_P2.50mm_Vertical, symbol PCM_SL_Connectors:JST_02
- added J5: Conn_01x04, Connector_PinHeader_2.54mm:PinHeader_1x04_P2.54mm_Vertical, symbol Connector_Generic:Conn_01x04
- added J6, J7: PINHD_1x2_Female, Connector_PinSocket_2.54mm:PinSocket_1x02_P2.54mm_Vertical, symbol PCM_SL_Pin_Headers:PINHD_1x2_Female
- added J8: PINHD_1x2_Female, TerminalBlock_Phoenix:TerminalBlock_Phoenix_MPT-0,5-2-2.54_1x02_P2.54mm_Horizontal, symbol PCM_SL_Pin_Headers:PINHD_1x2_Female
- added R10: 10k, LR0204F2K2:RESAD640W45L370D200, symbol LR0204F2K2:LR0204F2K2
- added R9: 220, LR0204F2K2:RESAD640W45L370D200, symbol LR0204F2K2:LR0204F2K2
- added U1: LM317T, PCM_Package_TO_SOT_THT_AKL:TO-220-3_Vertical, symbol PCM_Voltage_Regulator_AKL:LM317T
Connections:
- net RST_LORA is gone; now on net RST: RF1.4 (RST)
- net TIRQ is gone; now on net MISO: TOUCH1.4 (Pin_4)
- net +3.3V: now also CS1.3 (Pin_3), J6.1, J6.2, J7.1, J7.2, J8.1, U1.3 (IN); no longer RF1.3 (3.3V), SPI1.2 (Pin_2)
- net DC: now also CS1.2 (Pin_2); no longer CS1.3 (Pin_3)
- net GND: now also RF1.9 (GND), C3.2, J8.2, R10.2
- net MISO: now also SPI1.1 (Pin_1), SPI1.2 (Pin_2); no longer SPI1.3 (Pin_3), TOUCH1.3 (Pin_3)
- net MOSI: now also TOUCH1.3 (Pin_3); no longer CS1.4 (Pin_4)
- net RST: now also CS1.4 (Pin_4); no longer CS1.2 (Pin_2)
- net RX0: now also J3.1
- net RX2: now also J4.1
- net SCK: now also SPI1.3 (Pin_3); no longer SPI1.1 (Pin_1)
- net TX0: now also J3.2
- net TX2: now also J4.2
- net D33: now reaches DOIT1.22 (D33)
- net D33: now also J2.7
- net D25: now reaches DOIT1.23 (D25)
- net D25: now also J2.6
- net D26: now reaches DOIT1.24 (D26)
- net D26: now also J2.5
- net D27: now reaches DOIT1.25 (D27)
- net D27: now also J2.4
- net D14: now reaches DOIT1.26 (D14)
- net D14: now also J2.3
- net D12: now reaches DOIT1.27 (D12)
- net D12: now also J2.2
- net D13: now reaches DOIT1.28 (D13)
- net D13: now also J2.1
- net at RF1.8 (D103): now also J5.1 (Pin_1)
- net at RF1.7 (D102): now also J5.2 (Pin_2)
- net at RF1.6 (D101): now also J5.3 (Pin_3)
- net at RF1.5 (D100): now also J5.4 (Pin_4)
- new net: C3.1, R9.1, RF1.3 (3.3V), U1.2 (OUT)
- new net: R10.1, R9.2, U1.1
- no-connect marks 0 -> 1
Other:
- note removed: "NO CHIP SELECT PIN"
- moved on the sheet: C1

Commit message: final Update
Parts:
- removed 3.3vJ1: Conn_01x02, Connector_JST:JST_XH_B2B-XH-A_1x02_P2.50mm_Vertical, symbol Connector_Generic:Conn_01x02
- removed J8: PINHD_1x2_Female, TerminalBlock_Phoenix:TerminalBlock_Phoenix_MPT-0,5-2-2.54_1x02_P2.54mm_Horizontal, symbol PCM_SL_Pin_Headers:PINHD_1x2_Female
- removed R10: 10k, LR0204F2K2:RESAD640W45L370D200, symbol LR0204F2K2:LR0204F2K2
- added RV1: potentiometer_3362P, PCM_SL_Devices:potentiometer_3362P, symbol PCM_SL_Devices:potentiometer_3362P
Connections:
- net +5V: now also U1.3 (IN)
- net GND: now also J7.1, J7.2, RV1.1
- net 3v3: now reaches C3.1, R9.1, RF1.3 (3.3V), U1.2 (OUT)
- net 3v3: now also 3.3v1.2 (Pin_2), J6.1, J6.2, R5.2
- net at U1.1: now also RV1.2; no longer R9.2
- removed net +3.3V: 3.3v1.2 (Pin_2), CS1.3 (Pin_3), DOIT1.1 (3V3), J6.1, J6.2, J7.1, J7.2, R5.2, U1.3 (IN)
- new net: R9.2, RV1.3
- new net LED: CS1.3 (Pin_3), DOIT1.1 (3V3)
Other:
- moved on the sheet: R9
